File: AudioInjector.Octo.RCA.sch (KiCad schematic (older format))
At the start: 66 parts, among them P5 DAC_out, P6 ADC_in, U20 AV6-8.4-13, U21 AV8-8.4-13

Commit message: Fixed a bug in the output circuit. Updated part values.
Parts:
- C81, C82, C83, C84, C85, C86, C87, C88: value 3.3u -> 10u
- R46, R47, R48, R49, R54, R55, R56, R57: value 560 -> 562
Connections:
- net AOUT1+: now also C81.1; no longer C7.1, R46.2
- net AOUT2+: now also C82.1; no longer C8.1, R47.2
- net AOUT3+: now also C83.1; no longer C9.1, R48.2
- net AOUT4+: now also C84.1; no longer C10.1, R49.2
- net AOUT5+: now also C85.1; no longer C11.1, R54.2
- net AOUT6+: now also C86.1; no longer C12.1, R55.2
- net AOUT7+: now also C87.1; no longer C13.1, R56.2
- net AOUT8+: now also C88.1; no longer C14.1, R57.2
- net Out1: now also C7.1, R46.2; no longer C81.1
- net Out2: now also C8.1, R47.2; no longer C82.1
- net Out3: now also C9.1, R48.2; no longer C83.1
- net Out4: now also C10.1, R49.2; no longer C84.1
- net Out5: now also C11.1, R54.2; no longer C85.1
- net Out6: now also C12.1, R55.2; no longer C86.1
- net Out7: now also C13.1, R56.2; no longer C87.1
- net Out8: now also C14.1, R57.2; no longer C88.1
Changed lines of the file:
@@
 LIBS:contrib
 LIBS:valves
+LIBS:cs4270
+LIBS:spice
+LIBS:ak8111
+LIBS:mk1413
+LIBS:74hc_hct4040
+LIBS:sy10-100el3x
+LIBS:rca_double
+LIBS:dsc1001
+LIBS:adau1701
+LIBS:wm8581
+LIBS:Lattice_iCE_FPGA
+LIBS:wm8580
+LIBS:cs42448
+LIBS:fxo-hc73
+LIBS:lme49724
 LIBS:av8-8
+LIBS:PiMultiChannel-cache
 EELAYER 25 0
 EELAYER END
 $Descr A4 11693 8268
 encoding utf-8
-Sheet 1 1
+Sheet 2 2
 Title "Audio Injector Octo RCA breakout"
 Date ""
 Rev ""
-Comp "Flatmax"
-Comment1 "Single ended breakout"
-Comment2 "for the AudioInjector.net"
-Comment3 "Octo sound card for the Pi"
+Comp "Flatmax Pty Ltd"
+Comment1 "http://audioinjector.net"
+Comment2 "Single ended breakout"
+Comment3 ""
 Comment4 ""
 $EndDescr
@@
 P 8700 2850
 F 0 "R46" V 8780 2850 50  0000 C CNN
-F 1 "560" V 8700 2850 50  0000 C CNN
+F 1 "562" V 8700 2850 50  0000 C CNN
 F 2 "Resistors_SMD:R_0603" V 8630 2850 50  0001 C CNN
 F 3 "" H 8700 2850 50  0000 C CNN
@@
 P 9150 2850
 F 0 "C81" H 9265 2896 50  0000 L CNN
-F 1 "3.3u" H 9265 2804 50  0000 L CNN
+F 1 "10u" H 9265 2804 50  0000 L CNN
 F 2 "Capacitors_SMD:c_elec_5x5.3" H 9188 2700 50  0001 C CNN
 F 3 "" H 9150 2850 50  0000 C CNN
@@
 Text Label 7350 900  1    60   ~ 0
 Out8
+Text Label 8550 2850 2    60   ~ 0
+Out1
 Text Label 9300 2850 0    60   ~ 0
-Out1
-Text Label 8550 2850 2    60   ~ 0
 AOUT1+
 $Comp
@@
 P 8700 3300
 F 0 "R47" V 8780 3300 50  0000 C CNN
-F 1 "560" V 8700 3300 50  0000 C CNN
+F 1 "562" V 8700 3300 50  0000 C CNN
 F 2 "Resistors_SMD:R_0603" V 8630 3300 50  0001 C CNN
 F 3 "" H 8700 3300 50  0000 C CNN
@@
 P 9150 3300
 F 0 "C82" H 9265 3346 50  0000 L CNN
-F 1 "3.3u" H 9265 3254 50  0000 L CNN
+F 1 "10u" H 9265 3254 50  0000 L CNN
 F 2 "Capacitors_SMD:c_elec_5x5.3" H 9188 3150 50  0001 C CNN
 F 3 "" H 9150 3300 50  0000 C CNN
@@
 	8850 3300 9000 3300
 Connection ~ 8900 3300
+Text Label 8550 3300 2    60   ~ 0
+Out2
 Text Label 9300 3300 0    60   ~ 0
-Out2
-Text Label 8550 3300 2    60   ~ 0
 AOUT2+
 $Comp
@@
 P 8700 3750
 F 0 "R48" V 8780 3750 50  0000 C CNN
-F 1 "560" V 8700 3750 50  0000 C CNN
+F 1 "562" V 8700 3750 50  0000 C CNN
 F 2 "Resistors_SMD:R_0603" V 8630 3750 50  0001 C CNN
 F 3 "" H 8700 3750 50  0000 C CNN
@@
 P 9150 3750
 F 0 "C83" H 9265 3796 50  0000 L CNN
-F 1 "3.3u" H 9265 3704 50  0000 L CNN
+F 1 "10u" H 9265 3704 50  0000 L CNN
 F 2 "Capacitors_SMD:c_elec_5x5.3" H 9188 3600 50  0001 C CNN
 F 3 "" H 9150 3750 50  0000 C CNN
@@
 	8850 3750 9000 3750
 Connection ~ 8900 3750
+Text Label 8550 3750 2    60   ~ 0
+Out3
 Text Label 9300 3750 0    60   ~ 0
-Out3
-Text Label 8550 3750 2    60   ~ 0
 AOUT3+
 $Comp
@@
 P 8700 4200
 F 0 "R49" V 8780 4200 50  0000 C CNN
-F 1 "560" V 8700 4200 50  0000 C CNN
+F 1 "562" V 8700 4200 50  0000 C CNN
 F 2 "Resistors_SMD:R_0603" V 8630 4200 50  0001 C CNN
 F 3 "" H 8700 4200 50  0000 C CNN
@@
 P 9150 4200
 F 0 "C84" H 9265 4246 50  0000 L CNN
-F 1 "3.3u" H 9265 4154 50  0000 L CNN
+F 1 "10u" H 9265 4154 50  0000 L CNN
 F 2 "Capacitors_SMD:c_elec_5x5.3" H 9188 4050 50  0001 C CNN
 F 3 "" H 9150 4200 50  0000 C CNN
@@
 	8850 4200 9000 4200
 Connection ~ 8900 4200
+Text Label 8550 4200 2    60   ~ 0
+Out4
 Text Label 9300 4200 0    60   ~ 0
-Out4
-Text Label 8550 4200 2    60   ~ 0
 AOUT4+
 $Comp
@@
 P 10200 2850
 F 0 "R54" V 10280 2850 50  0000 C CNN
-F 1 "560" V 10200 2850 50  0000 C CNN
+F 1 "562" V 10200 2850 50  0000 C CNN
 F 2 "Resistors_SMD:R_0603" V 10130 2850 50  0001 C CNN
 F 3 "" H 10200 2850 50  0000 C CNN
@@
 P 10650 2850
 F 0 "C85" H 10765 2896 50  0000 L CNN
-F 1 "3.3u" H 10765 2804 50  0000 L CNN
+F 1 "10u" H 10765 2804 50  0000 L CNN
 F 2 "Capacitors_SMD:c_elec_5x5.3" H 10688 2700 50  0001 C CNN
 F 3 "" H 10650 2850 50  0000 C CNN
@@
 	10350 2850 10500 2850
 Connection ~ 10400 2850
+Text Label 10050 2850 2    60   ~ 0
+Out5
 Text Label 10800 2850 0    60   ~ 0
-Out5
-Text Label 10050 2850 2    60   ~ 0
 AOUT5+
 $Comp
@@
 P 10200 3300
 F 0 "R55" V 10280 3300 50  0000 C CNN
-F 1 "560" V 10200 3300 50  0000 C CNN
+F 1 "562" V 10200 3300 50  0000 C CNN
 F 2 "Resistors_SMD:R_0603" V 10130 3300 50  0001 C CNN
 F 3 "" H 10200 3300 50  0000 C CNN
@@
 P 10650 3300
 F 0 "C86" H 10765 3346 50  0000 L CNN
-F 1 "3.3u" H 10765 3254 50  0000 L CNN
+F 1 "10u" H 10765 3254 50  0000 L CNN
 F 2 "Capacitors_SMD:c_elec_5x5.3" H 10688 3150 50  0001 C CNN
 F 3 "" H 10650 3300 50  0000 C CNN
@@
 	10350 3300 10500 3300
 Connection ~ 10400 3300
+Text Label 10050 3300 2    60   ~ 0
+Out6
 Text Label 10800 3300 0    60   ~ 0
-Out6
-Text Label 10050 3300 2    60   ~ 0
 AOUT6+
 $Comp
@@
 P 10200 3750
 F 0 "R56" V 10280 3750 50  0000 C CNN
-F 1 "560" V 10200 3750 50  0000 C CNN
+F 1 "562" V 10200 3750 50  0000 C CNN
 F 2 "Resistors_SMD:R_0603" V 10130 3750 50  0001 C CNN
 F 3 "" H 10200 3750 50  0000 C CNN
@@
 P 10650 3750
 F 0 "C87" H 10765 3796 50  0000 L CNN
-F 1 "3.3u" H 10765 3704 50  0000 L CNN
+F 1 "10u" H 10765 3704 50  0000 L CNN
 F 2 "Capacitors_SMD:c_elec_5x5.3" H 10688 3600 50  0001 C CNN
 F 3 "" H 10650 3750 50  0000 C CNN
@@
 	10350 3750 10500 3750
 Connection ~ 10400 3750
+Text Label 10050 3750 2    60   ~ 0
+Out7
 Text Label 10800 3750 0    60   ~ 0
-Out7
-Text Label 10050 3750 2    60   ~ 0
 AOUT7+
 $Comp
@@
 P 10200 4200
 F 0 "R57" V 10280 4200 50  0000 C CNN
-F 1 "560" V 10200 4200 50  0000 C CNN
+F 1 "562" V 10200 4200 50  0000 C CNN
 F 2 "Resistors_SMD:R_0603" V 10130 4200 50  0001 C CNN
 F 3 "" H 10200 4200 50  0000 C CNN
@@
 P 10650 4200
 F 0 "C88" H 10765 4246 50  0000 L CNN
-F 1 "3.3u" H 10765 4154 50  0000 L CNN
+F 1 "10u" H 10765 4154 50  0000 L CNN
 F 2 "Capacitors_SMD:c_elec_5x5.3" H 10688 4050 50  0001 C CNN
 F 3 "" H 10650 4200 50  0000 C CNN
@@
 	10350 4200 10500 4200
 Connection ~ 10400 4200
+Text Label 10050 4200 2    60   ~ 0
+Out8
 Text Label 10800 4200 0    60   ~ 0
-Out8
-Text Label 10050 4200 2    60   ~ 0
 AOUT8+
 Text Label 6200 4300 1    60   ~ 0

Commit message: Adding v1.5 of these PCBs.
Connections:
- net ADC_fb1+: now also P6.4 (P4); no longer P6.3 (P3)
- net ADC_fb1-: now also P6.2 (P2); no longer P6.1 (P1)
- net ADC_fb2+: now also P6.8 (P8); no longer P6.7 (P7)
- net ADC_fb2-: now also P6.6 (P6); no longer P6.5 (P5)
- net ADC_fb3+: now also P6.12 (P12); no longer P6.11 (P11)
- net ADC_fb3-: now also P6.10 (P10); no longer P6.9 (P9)
- net ADC_fb4+: now also P6.16 (P16); no longer P6.15 (P15)
- net ADC_fb4-: now also P6.14 (P14); no longer P6.13 (P13)
- net ADC_fb5+: now also P6.20 (P20); no longer P6.19 (P19)
- net ADC_fb5-: now also P6.18 (P18); no longer P6.17 (P17)
- net ADC_fb6+: now also P6.24 (P24); no longer P6.23 (P23)
- net ADC_fb6-: now also P6.22 (P22); no longer P6.21 (P21)
- net AGND: now also P5.3 (P3), P6.11 (P11), P6.13 (P13), P6.15 (P15), P6.17 (P17), P6.19 (P19), P6.5 (P5), P6.7 (P7), P6.9 (P9); no longer P5.4 (P4), P6.10 (P10), P6.12 (P12), P6.14 (P14), P6.16 (P16), P6.18 (P18), P6.20 (P20), P6.6 (P6), P6.8 (P8)
- net AOUT1+: now also P5.17 (P17); no longer P5.18 (P18)
- net AOUT1-: now also P5.19 (P19); no longer P5.20 (P20)
- net AOUT2+: now also P5.20 (P20); no longer P5.19 (P19)
- net AOUT2-: now also P5.18 (P18); no longer P5.17 (P17)
- net AOUT3+: now also P5.13 (P13); no longer P5.14 (P14)
- net AOUT3-: now also P5.15 (P15); no longer P5.16 (P16)
- net AOUT4+: now also P5.16 (P16); no longer P5.15 (P15)
- net AOUT4-: now also P5.14 (P14); no longer P5.13 (P13)
- net AOUT5+: now also P5.9 (P9); no longer P5.10 (P10)
- net AOUT5-: now also P5.11 (P11); no longer P5.12 (P12)
- net AOUT6+: now also P5.12 (P12); no longer P5.11 (P11)
- net AOUT6-: now also P5.10 (P10); no longer P5.9 (P9)
- net AOUT7+: now also P5.5 (P5); no longer P5.6 (P6)
- net AOUT7-: now also P5.7 (P7); no longer P5.8 (P8)
- net AOUT8+: now also P5.8 (P8); no longer P5.7 (P7)
- net AOUT8-: now also P5.6 (P6); no longer P5.5 (P5)
- net MUTEC: now also P5.4 (P4); no longer P5.3 (P3)
- net V5: now also P6.1 (P1), P6.21 (P21), P6.23 (P23), P6.3 (P3); no longer P6.2 (P2), P6.22 (P22), P6.24 (P24), P6.4 (P4)
Changed lines of the file:
@@
 LIBS:valves
 LIBS:cs4270
-LIBS:spice
 LIBS:ak8111
 LIBS:mk1413
@@
 LIBS:wm8581
 LIBS:Lattice_iCE_FPGA
-LIBS:wm8580
 LIBS:cs42448
 LIBS:fxo-hc73
@@
 F 3 "" H 5250 3350 50  0000 C CNN
 	1    5250 4550
-	0    1    -1   0
+	0    1    1    0
 $EndComp
 $Comp
@@
 F 3 "" H 6650 3350 50  0000 C CNN
 	1    6650 4550
-	0    1    1    0
+	0    1    -1   0
 $EndComp
 $Comp
